File: design/_autosave-BLDC_4_old.kicad_pcb (KiCad board)
At the start: 4 copper layers, 38.5 x 65 mm, 129 parts, among them K1 SERVO, P1 HALL/Encoder, P101 CANBUS, P2 SWD, P3 PWR_COMM, P4 IN+, P5 IN-, P6 MOTOR1, P7 MOTOR2, P9 MOTOR3, Q1 IRFS3006, Q2 IRFS3006, Q3 IRFS3006, Q4 IRFS3006, Q5 IRFS3006, Q6 IRFS3006, U1 STM32F40X_LQFP64, U2 NCP1117ST33T3G, U3 DRV8302, U401 SN65HVD232, X1 MINI-USB-SHIELD-32005-201, X2 8MHz 10ppm

Commit message: More layouting
Changed lines of the file:
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@@
-(kicad_pcb (version 4) (host pcbnew "(2015-02-11 BZR 5414)-product")
+(kicad_pcb (version 4) (host pcbnew "(2015-03-02 BZR 5466)-product")
   (general
     (links 308)
     (no_connects 0)
-    (area 77.3847 78.682 118.339914 145.81)
+    (area 78.424999 79.924999 117.075001 145.075001)
     (thickness 1.6)
     (drawings 32)
-    (tracks 1799)
+    (tracks 1800)
     (zones 0)
     (modules 129)
@@
   )
   (layers
-    (0 F.Cu signal hide)
+    (0 F.Cu signal)
     (1 GND signal hide)
     (2 Power signal hide)
-    (31 B.Cu signal)
-    (32 B.Adhes user hide)
-    (33 F.Adhes user hide)
+    (31 B.Cu signal hide)
+    (32 B.Adhes user)
+    (33 F.Adhes user)
     (34 B.Paste user hide)
-    (35 F.Paste user hide)
-    (36 B.SilkS user hide)
-    (37 F.SilkS user hide)
-    (38 B.Mask user hide)
+    (35 F.Paste user)
+    (36 B.SilkS user)
+    (37 F.SilkS user)
+    (38 B.Mask user)
     (39 F.Mask user hide)
     (40 Dwgs.User user hide)
-    (41 Cmts.User user hide)
-    (42 Eco1.User user hide)
-    (43 Eco2.User user hide)
-    (44 Edge.Cuts user hide)
+    (41 Cmts.User user)
+    (42 Eco1.User user)
+    (43 Eco2.User user)
+    (44 Edge.Cuts user)
   )
   (setup
@@
     (pad_to_mask_clearance 0)
     (aux_axis_origin 0 0)
-    (visible_elements 7FFF3E3F)
+    (visible_elements 7FFD7E6B)
     (pcbplotparams
       (layerselection 0x00030_80000001)
@@
   )
   (gr_line (start 117 80) (end 78.5 80) (angle 90) (layer Edge.Cuts) (width 0.15))
+  (segment (start 89.67 123.26) (end 89.69 123.24) (width 0.2032) (layer F.Cu) (net 0))
   (segment (start 114.3 118.03126) (end 114.3 119.634) (width 1.016) (layer Power) (net 1) (status 10))
   (segment (start 112.395 133.858) (end 111.252 135.001) (width 1.016) (layer Power) (net 1) (status 20))
@@
   (segment (start 108.839 131.699) (end 106.553 131.699) (width 0.254) (layer B.Cu) (net 45))
   (segment (start 111.475185 129.824815) (end 110.713185 129.824815) (width 0.254) (layer B.Cu) (net 45))
-  (segment (start 99.695 107.6325) (end 99.695 109.22) (width 0.3048) (layer F.Cu) (net 46) (status 10))
-  (segment (start 100.1395 107.188) (end 99.695 107.6325) (width 0.3048) (layer F.Cu) (net 46) (status 30))
-  (segment (start 99.695 109.22) (end 99.695 110.236) (width 0.3048) (layer F.Cu) (net 46))
-  (segment (start 99.695 110.236) (end 100.15728 110.69828) (width 0.3048) (layer F.Cu) (net 46))
   (segment (start 90.79 85.71) (end 105.776 85.71) (width 0.635) (layer Power) (net 46))
   (segment (start 105.776 85.71) (end 106.934 86.868) (width 0.635) (layer Power) (net 46))
@@
   (via (at 110.744 90.424) (size 1.524) (drill 0.762) (layers F.Cu B.Cu) (net 46) (status 30))
   (via (at 112.522 90.424) (size 1.524) (drill 0.762) (layers F.Cu B.Cu) (net 46) (status 30))
+  (segment (start 99.695 107.6325) (end 99.695 109.22) (width 0.3048) (layer F.Cu) (net 46) (status 10))
   (via (at 99.695 109.22) (size 0.8) (drill 0.5) (layers F.Cu B.Cu) (net 46))
+  (segment (start 100.1395 107.188) (end 99.695 107.6325) (width 0.3048) (layer F.Cu) (net 46) (status 30))
   (segment (start 100.15728 111.8235) (end 100.15728 110.69828) (width 0.3048) (layer F.Cu) (net 46) (status 10))
+  (segment (start 99.695 110.236) (end 100.15728 110.69828) (width 0.3048) (layer F.Cu) (net 46))
+  (segment (start 99.695 109.22) (end 99.695 110.236) (width 0.3048) (layer F.Cu) (net 46))
   (segment (start 109.474 82.804) (end 109.474 87.24646) (width 0.254) (layer F.Cu) (net 46) (status 30))
   (segment (start 108.966 83.312) (end 109.474 82.804) (width 2.286) (layer F.Cu) (net 46) (status 30))
@@
   (segment (start 97.917 125.603) (end 93.599 125.603) (width 0.254) (layer Power) (net 78))
   (segment (start 98.85 126.65) (end 97.917 125.603) (width 0.254) (layer Power) (net 78))
-  (segment (start 85.40426 138.504) (end 100.256 138.504) (width 0.254) (layer F.Cu) (net 79))
   (segment (start 85.40426 138.504) (end 84.10026 137.2) (width 0.254) (layer F.Cu) (net 79) (status 20))
   (segment (start 81.788 135.128) (end 83.312 135.128) (width 0.254) (layer B.Cu) (net 79) (status 30))
@@
   (segment (start 100.256 138.504) (end 100.58908 138.17092) (width 0.254) (layer F.Cu) (net 79))
   (segment (start 100.58908 138.17092) (end 100.58908 136.81456) (width 0.254) (layer F.Cu) (net 79) (status 20))
+  (segment (start 85.40426 138.504) (end 100.256 138.504) (width 0.254) (layer F.Cu) (net 79))
   (segment (start 92.456 132.588) (end 92.456 133.604) (width 0.254) (layer B.Cu) (net 80) (status 30))
   (segment (start 95.08744 128.81356) (end 94.234 128.81356) (width 0.2032) (layer F.Cu) (net 80) (status 10))
